File: USBtiny_custom.sch (KiCad schematic (older format))
At the start: 28 parts, among them J1 USB_B_Micro, J2 USB_A, J3 AVR-ISP-6, SW1 SW_SPDT, U1 ATtiny2313-20SU, U2 74125, Y1 12M

Commit message: kicad meta update
Parts:
- gave numbers to parts that had none: 1
Changed lines of the file:
@@
 NoConn ~ 5200 6000
 $Comp
-L Connector:TestPoint_Flag TP?
+L Connector:TestPoint_Flag TP1
 U 1 1 5C460011
 P 950 2400
-F 0 "TP?" H 910 2403 50  0000 R CNN
+F 0 "TP1" H 910 2403 50  0000 R CNN
 F 1 "TestPoint_Flag" H 1300 2600 50  0000 R CNN
 F 2 "TestPoint:TestPoint_Pad_1.5x1.5mm" H 1150 2400 50  0001 C CNN
